File: pcb/djiFriend.kicad_pcb (KiCad board)
At the start: 2 copper layers, 76.9 x 38.8 mm, 46 parts, among them J1 Batt, J2 USB_B_Micro, J4 AVR-ISP-6, Q1 BSS84W, SW1 FSMRA4JH04, SW2 INPUT, U1 AP1117-50, U2 MT3608, U3 ATmega328P-A, U4 BQ24005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

Commit message: added gerbers, updated version numbers
Other:
- board text added: "djiFriend v1.1"
- board text removed: "djiFriend v1.0"
Changed lines of the file:
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@@
     (effects (font (size 1.143 1.143) (thickness 0.2032)))
   )
-  (gr_text "djiFriend v1.0" (at 70.7566 78.2916 90) (layer "F.SilkS")
+  (gr_text "djiFriend v1.1" (at 70.756602 78.291588 90) (layer "F.SilkS")
     (effects (font (size 1.143 1.143) (thickness 0.2032)))
   )
