File: pcb/djiFriend.kicad_sch (KiCad schematic)
At the start: 46 parts, among them J1 Batt, J2 USB_B_Micro, J4 AVR-ISP-6, Q1 BSS84W, SW1 FSMRA4JH04, SW2 INPUT, U1 AP1117-50, U2 MT3608, U3 ATmega328P-A, U4 BQ24005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

Commit message: added gerbers, updated version numbers
Other:
- title: DJI Battery Friend -> DJI Friend
Changed lines of the file:
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@@
   (paper "A4")
   (title_block
-    (title "DJI Battery Friend")
-    (date "2022-08-25")
-    (rev "v01")
-    (comment 1 "Licence:")
+    (title "DJI Friend")
+    (date "2022-10-17")
+    (rev "v1.1")
     (comment 3 "github.com/theloukou")
     (comment 4 "Author: Lefteris Kantakos")
